File: E70N19_Dev_Board/E70N19_Dev_Board.kicad_pcb (KiCad board)
At the start: 2 copper layers, 0 parts

Commit message: Finishing PCB component placement
Parts:
- added C1: 4.7uF, Capacitors_SMD:C_0603, F.Cu at (115.6, 38.1)
- added C10: 100nF, Capacitors_SMD:C_0603, F.Cu at (133.9, 81.3)
- added C11: 100nF, Capacitors_SMD:C_0603, F.Cu at (135.1, 61.0)
- added C12: 100nF, Capacitors_SMD:C_0603, F.Cu at (124.5, 56.6)
- added C13: 100nF, Capacitors_SMD:C_0603, F.Cu at (117.6, 76.2)
- added C14: 1uF, Capacitors_SMD:C_0603, F.Cu at (115.0, 72.4)
- added C15: 100nF, Capacitors_SMD:C_0603, F.Cu at (115.0, 73.7)
- added C16: 100nF, Capacitors_SMD:C_0603, F.Cu at (120.7, 81.8)
- added C17: 100nF, Capacitors_SMD:C_0603, F.Cu at (123.2, 81.8)
- added C18: 100nF, Capacitors_SMD:C_0603, F.Cu at (138.9, 77.5)
- added C19: 100nF, Capacitors_SMD:C_0603, F.Cu at (125.7, 56.6)
- added C2: 10uF, Capacitors_SMD:C_0805, F.Cu at (93.0, 37.8)
- added C20: 100nF, Capacitors_SMD:C_0603, F.Cu at (121.9, 57.9)
- added C21: 100nF, Capacitors_SMD:C_0603, F.Cu at (118.1, 65.3)
- added C22: 10pF, Capacitors_SMD:C_0603, F.Cu at (116.8, 65.3)
- added C23: 18pF, Capacitors_SMD:C_0603, F.Cu at (111.8, 69.1)
- added C24: 18pF, Capacitors_SMD:C_0603, F.Cu at (113.0, 66.0)
- added C25: 1uF, Capacitors_SMD:C_0603, F.Cu at (171.4, 97.0)
- added C26: 100nF, Capacitors_SMD:C_0603, F.Cu at (101.1, 109.2)
- added C27: 10uF, Capacitors_SMD:C_0805, F.Cu at (175.3, 110.5)
- added C28: 100nF, Capacitors_SMD:C_0603, F.Cu at (118.6, 78.7)
- added C29: 100nF, Capacitors_SMD:C_0603, F.Cu at (102.9, 50.8)
- added C3: 4.7uF, Capacitors_SMD:C_0603, F.Cu at (118.1, 40.6)
- added C30: 10nF, Capacitors_SMD:C_0603, F.Cu at (100.8, 58.4)
- added C31: 12.5pF, Capacitors_SMD:C_0603, F.Cu at (123.7, 86.4)
- added C32: 12.5pF, Capacitors_SMD:C_0603, F.Cu at (128.8, 86.4)
- added C4: 0.1uF, Capacitors_SMD:C_0603, F.Cu at (105.4, 47.0)
- added C5: 10uF, Capacitors_SMD:C_0805, F.Cu at (101.6, 63.5)
- added C6: 4.7uF, Capacitors_SMD:C_0603, F.Cu at (118.1, 53.9)
- added C7: 100nF, Capacitors_SMD:C_0603, F.Cu at (120.7, 57.9)
- added C8: 100nF, Capacitors_SMD:C_0603, F.Cu at (119.4, 57.9)
- added C9: 100nF, Capacitors_SMD:C_0603, F.Cu at (121.9, 81.8)
- added D1: LED, LEDs:LED_0805, F.Cu at (120.8, 44.5)
- added D2: LED, LEDs:LED_0805, F.Cu at (171.6, 113.0)
- added D3: LED, LEDs:LED_0805, F.Cu at (94.2, 53.3)
- added FP1: BM71BLES1FC2, eclectronics:BM71BLES1FC2, F.Cu at (178.7, 99.2)
- added J1: USB_microB_2040002-1, eclectronics:USB_microB_2040002-1, F.Cu at (88.7, 31.8)
- added J2: Battery 1x2, Connectors_JST:JST_PH_S2B-PH-SM4-TB_02x2.00mm_Angled, F.Cu at (104.1, 35.6)
- added J3: JTAGSEL_JUMPER 1x3, Pin_Headers:Pin_Header_Straight_1x03_Pitch2.54mm, F.Cu at (129.5, 40.6)
- added J4: UART_PROG 1x2, Pin_Headers:Pin_Header_Straight_1x02_Pitch2.54mm, F.Cu at (171.4, 35.6)
- added J5: ERASE_JUMPER 1x3, Pin_Headers:Pin_Header_Straight_1x03_Pitch2.54mm, F.Cu at (160.0, 40.6)
- added J6: ARM-Cortex-Debug-10, Pin_Headers:Pin_Header_Straight_2x05_Pitch2.54mm, F.Cu at (142.2, 40.6)
- added J7: CAN 1x2, Pin_Headers:Pin_Header_Straight_1x02_Pitch2.54mm, F.Cu at (94.0, 106.7)
- added J8: Conn_02x15_Counter_Clockwise, Pin_Headers:Pin_Header_Straight_2x15_Pitch2.54mm, F.Cu at (77.5, 64.8)
- added J9: Conn_02x15_Counter_Clockwise, Pin_Headers:Pin_Header_Straight_2x15_Pitch2.54mm, F.Cu at (184.2, 48.3)
- added L1: 470R @ 100MHz, Resistors_SMD:R_0603, F.Cu at (121.9, 52.6)
- added L2: 470R @ 100MHz, Resistors_SMD:R_0603, F.Cu at (114.3, 57.7)
- added R1: 475, Resistors_SMD:R_0603, F.Cu at (122.4, 40.6)
- added R10: 100K, Resistors_SMD:R_0603, F.Cu at (143.5, 33.0)
- added R11: 100K, Resistors_SMD:R_0603, F.Cu at (151.9, 33.0)
- added R12: 63.4, Resistors_SMD:R_0603, F.Cu at (113.0, 61.7)
- added R13: 1K, Resistors_SMD:R_0603, F.Cu at (94.0, 55.9)
- added R14: 30, Resistors_SMD:R_0603, F.Cu at (90.2, 38.9)
- added R15: 30, Resistors_SMD:R_0603, F.Cu at (87.6, 38.9)
- added R2: 402, Resistors_SMD:R_0603, F.Cu at (91.4, 49.5)
- added R3: 2K, Resistors_SMD:R_0603, F.Cu at (114.3, 47.0)
- added R4: 4.99K, Resistors_SMD:R_0603, F.Cu at (115.6, 61.5)
- added R5: 4.75K, Resistors_SMD:R_0603, F.Cu at (177.8, 95.2)
- added R6: 10K, Resistors_SMD:R_0603, F.Cu at (86.9, 49.5)
- added R7: 20K, Resistors_SMD:R_0603, F.Cu at (90.7, 47.0)
- added R8: 402, Resistors_SMD:R_0603, F.Cu at (170.7, 108.0)
- added R9: 100K, Resistors_SMD:R_0603, F.Cu at (148.6, 33.0)
- added SW1: NRST_BUTTON, eclectronics:PTS820_J15M_SMTR_LFS, F.Cu at (147.7, 49.5)
- added U1: MCP73831, TO_SOT_Packages_SMD:SOT-23-5, F.Cu at (114.5, 42.2)
- added U2: TPS2112A, Housings_SSOP:TSSOP-8_4.4x3mm_Pitch0.65mm, F.Cu at (99.1, 47.0)
- added U3: SPX3819M5-L-3-3, TO_SOT_Packages_SMD:SOT-23-5, F.Cu at (97.6, 62.5)
- added U4: ATSAME70N19, Housings_QFP:LQFP-100_14x14mm_Pitch0.5mm, F.Cu at (129.0, 70.7)
- added U5: RT9818A-18GV, TO_SOT_Packages_SMD:SOT-23, F.Cu at (167.6, 98.1)
- added U6: SN65HVD233-Q1, Housings_SOIC:SOIC-8_3.9x4.9mm_Pitch1.27mm, F.Cu at (105.6, 103.5)
- added Y1: Crystal_Small, eclectronics:ECS-.327-12.5-34B-TR, F.Cu at (124.6, 83.8)
- added Y2: Crystal, Crystals:Crystal_SMD_SeikoEpson_FA238-4pin_3.2x2.5mm, F.Cu at (115.4, 68.6)
Other:
- net class Default: clearance 0.2 -> 0.1524; trace_width 0.25 -> 0.1524; via_dia 0.6 -> 0.5842; via_drill 0.4 -> 0.4064
- rule trace_clearance: 0.2 -> 0.1524
- rule trace_min: 0.2 -> 0.1524
- rule via_min_size: 0.4 -> 0.4064
