File: E70N19_Dev_Board/E70N19_Dev_Board.sch (KiCad schematic (older format))
At the start: 77 parts, among them J1 USB_microB_2040002-1, J2 Battery 1x2, J3 JTAGSEL_JUMPER 1x3, J4 UART_PROG 1x2, J5 ERASE_JUMPER 1x3, J6 ARM-Cortex-Debug-10, J7 CAN 1x2, J8 Conn_02x15_Counter_Clockwise, J9 Conn_02x15_Counter_Clockwise, SW1 NRST_BUTTON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

Commit message: Fixed up fanout connections
Connections:
- net GND: now also J9.6 (Pin_6)
- net PA5: no longer J9.6 (Pin_6)
Changed lines of the file:
@@
 	1    0    0    -1
 $EndComp
-Text Label 15325 6650 2    60   ~ 0
-PA5
 Text Label 15325 6550 2    60   ~ 0
 PD11
@@
 Text Label 15325 7450 2    60   ~ 0
 PD17
-Text Label 15325 7550 2    60   ~ 0
-PA5
 Text Label 15825 7550 0    60   ~ 0
 PA27
@@
 Text Label 15825 6150 0    60   ~ 0
 PA23
+$Comp
+L GND #PWR055
+U 1 1 59E0B7E1
+P 15000 6675
+F 0 "#PWR055" H 15000 6425 50  0001 C CNN
+F 1 "GND" H 15000 6525 50  0000 C CNN
+F 2 "" H 15000 6675 50  0000 C CNN
+F 3 "" H 15000 6675 50  0000 C CNN
+	1    15000 6675
+	1    0    0    -1
+$EndComp
+Wire Wire Line
+	15325 6650 15000 6650
+Wire Wire Line
+	15000 6650 15000 6675
+Text Label 15325 7550 2    60   ~ 0
+PA5
 $EndSCHEMATC
